Commit message: Add yajun's experiments

File: iiwa_description/urdf/iiwa.gazebo.xacro (robot description, xacro)
@@ -2,16 +2,4 @@
 <robot xmlns:xacro="http://www.ros.org/wiki/xacro">
   <xacro:macro name="iiwa_gazebo" params="robot_name">
-     <!-- Enable the Joint Feedback -->
-    <gazebo reference="${robot_name}_joint_7">
-      <provideFeedback>true</provideFeedback>
-    </gazebo>
-    <!-- The ft_sensor plugin -->
-    <gazebo>
-      <plugin name="ft_sensor" filename="libgazebo_ros_ft_sensor.so">
-        <updateRate>50.0</updateRate>
-        <topicName>/${robot_name}/state/CartesianWrench</topicName>
-        <jointName>${robot_name}_joint_7</jointName>
-      </plugin>
-    </gazebo>
     <!-- Load Gazebo lib and set the robot namespace -->
     <gazebo>

File: iiwa_description/urdf/iiwa.transmission.xacro (robot description, xacro)
@@ -6,9 +6,9 @@
       <type>transmission_interface/SimpleTransmission</type>
       <joint name="${robot_name}_joint_1">
-        <hardwareInterface>hardware_interface/${hardware_interface}</hardwareInterface>
+	<hardwareInterface>${hardware_interface}</hardwareInterface>
       </joint>
       <actuator name="${robot_name}_motor_1">
-        <hardwareInterface>hardware_interface/${hardware_interface}</hardwareInterface>
-        <mechanicalReduction>1</mechanicalReduction>
+	<hardwareInterface>${hardware_interface}</hardwareInterface>
+	<mechanicalReduction>1</mechanicalReduction>
       </actuator>
     </transmission>
@@ -17,9 +17,9 @@
       <type>transmission_interface/SimpleTransmission</type>
       <joint name="${robot_name}_joint_2">
-        <hardwareInterface>hardware_interface/${hardware_interface}</hardwareInterface>
+	<hardwareInterface>${hardware_interface}</hardwareInterface>
       </joint>
       <actuator name="${robot_name}_motor_2">
-        <hardwareInterface>hardware_interface/${hardware_interface}</hardwareInterface>
-        <mechanicalReduction>1</mechanicalReduction>
+	<hardwareInterface>${hardware_interface}</hardwareInterface>
+	<mechanicalReduction>1</mechanicalReduction>
       </actuator>
     </transmission>
@@ -28,9 +28,9 @@
       <type>transmission_interface/SimpleTransmission</type>
       <joint name="${robot_name}_joint_3">
-        <hardwareInterface>hardware_interface/${hardware_interface}</hardwareInterface>
+	<hardwareInterface>${hardware_interface}</hardwareInterface>
       </joint>
       <actuator name="${robot_name}_motor_3">
-        <hardwareInterface>hardware_interface/${hardware_interface}</hardwareInterface>
-        <mechanicalReduction>1</mechanicalReduction>
+	<hardwareInterface>${hardware_interface}</hardwareInterface>
+	<mechanicalReduction>1</mechanicalReduction>
       </actuator>
     </transmission>
@@ -39,9 +39,9 @@
       <type>transmission_interface/SimpleTransmission</type>
       <joint name="${robot_name}_joint_4">
-        <hardwareInterface>hardware_interface/${hardware_interface}</hardwareInterface>
+	<hardwareInterface>${hardware_interface}</hardwareInterface>
       </joint>
       <actuator name="${robot_name}_motor_4">
-        <hardwareInterface>hardware_interface/${hardware_interface}</hardwareInterface>
-        <mechanicalReduction>1</mechanicalReduction>
+	<hardwareInterface>${hardware_interface}</hardwareInterface>
+	<mechanicalReduction>1</mechanicalReduction>
       </actuator>
     </transmission>
@@ -50,9 +50,9 @@
       <type>transmission_interface/SimpleTransmission</type>
       <joint name="${robot_name}_joint_5">
-        <hardwareInterface>hardware_interface/${hardware_interface}</hardwareInterface>
+	<hardwareInterface>${hardware_interface}</hardwareInterface>
       </joint>
       <actuator name="${robot_name}_motor_5">
-        <hardwareInterface>hardware_interface/${hardware_interface}</hardwareInterface>
-        <mechanicalReduction>1</mechanicalReduction>
+	<hardwareInterface>${hardware_interface}</hardwareInterface>
+	<mechanicalReduction>1</mechanicalReduction>
       </actuator>
     </transmission>
@@ -61,9 +61,9 @@
       <type>transmission_interface/SimpleTransmission</type>
       <joint name="${robot_name}_joint_6">
-        <hardwareInterface>hardware_interface/${hardware_interface}</hardwareInterface>
+	<hardwareInterface>${hardware_interface}</hardwareInterface>
       </joint>
       <actuator name="${robot_name}_motor_6">
-        <hardwareInterface>hardware_interface/${hardware_interface}</hardwareInterface>
-        <mechanicalReduction>1</mechanicalReduction>
+	<hardwareInterface>${hardware_interface}</hardwareInterface>
+	<mechanicalReduction>1</mechanicalReduction>
       </actuator>
     </transmission>
@@ -72,9 +72,9 @@
       <type>transmission_interface/SimpleTransmission</type>
       <joint name="${robot_name}_joint_7">
-        <hardwareInterface>hardware_interface/${hardware_interface}</hardwareInterface>
+	<hardwareInterface>${hardware_interface}</hardwareInterface>
       </joint>
       <actuator name="${robot_name}_motor_7">
-        <hardwareInterface>hardware_interface/${hardware_interface}</hardwareInterface>
-        <mechanicalReduction>1</mechanicalReduction>
+	<hardwareInterface>${hardware_interface}</hardwareInterface>
+	<mechanicalReduction>1</mechanicalReduction>
       </actuator>
     </transmission>

File: iiwa_description/urdf/iiwa7.xacro (robot description, xacro)
@@ -274,5 +274,5 @@
         <origin xyz="0 0 -0.0005" rpy="0 0 0"/>
         <geometry>
-          <mesh filename="package://iiwa_description/meshes/iiwa7/visual/link_7.stl"/>
+          <mesh filename="package://iiwa_description/meshes/iiwa7/visual/MF_Touch_pneumatisch.dae"/>
         </geometry>
         <material name="Grey"/>
@@ -281,5 +281,5 @@
         <origin xyz="0 0 -0.0005" rpy="0 0 0"/>
         <geometry>
-          <mesh filename="package://iiwa_description/meshes/iiwa7/collision/link_7.stl"/>
+          <mesh filename="package://iiwa_description/meshes/iiwa7/collision/MF_Touch_pneumatisch.dae"/>
         </geometry>
         <material name="Grey"/>
@@ -289,7 +289,28 @@
       <parent link="${robot_name}_link_7"/>
       <child link="${robot_name}_link_ee"/>
-      <origin xyz="0 0 0.045" rpy="0 0 0"/>
+      <origin xyz="0 0 0.071" rpy="0 0 0"/> <!--0.045-->
     </joint>
     <link name="${robot_name}_link_ee">
+    <visual>
+        <origin xyz="0 0 0" rpy="${PI / 2} 0 0"/>
+        <geometry>
+          <mesh filename="package://iiwa_description/meshes/iiwa7/visual/tool_pneumatisch.dae"/>
+        </geometry>
+        <material name="Grey"/>
+      </visual>
+      <collision>
+        <origin xyz="0 0 0" rpy="${PI / 2} 0 0"/>
+        <geometry>
+          <mesh filename="package://iiwa_description/meshes/iiwa7/collision/tool_pneumatisch.dae"/>
+        </geometry>
+        <material name="Grey"/>
+      </collision>
+    </link>
+    <joint name="${robot_name}_joint_tool" type="fixed">
+      <parent link="${robot_name}_link_ee"/>
+      <child link="${robot_name}_link_tool"/>
+      <origin xyz="0 0 0" rpy="${PI} 0 ${PI}"/>
+    </joint>
+    <link name="${robot_name}_link_tool">
     </link>
     <!--Extensions -->

Commit message: Add yajun's modification and support ros melodic

File: iiwa_description/urdf/iiwa.gazebo.xacro (robot description, xacro)
@@ -3,9 +3,9 @@
   <xacro:macro name="iiwa_gazebo" params="robot_name">
      <!-- Enable the Joint Feedback -->
-    <gazebo reference="${robot_name}_joint_7">
+    <!-- <gazebo reference="${robot_name}_joint_7">
       <provideFeedback>true</provideFeedback>
-    </gazebo>
+    </gazebo> -->
     <!-- The ft_sensor plugin -->
-    <gazebo>
+    <!-- <gazebo>
       <plugin name="ft_sensor" filename="libgazebo_ros_ft_sensor.so">
         <updateRate>50.0</updateRate>
@@ -13,5 +13,5 @@
         <jointName>${robot_name}_joint_7</jointName>
       </plugin>
-    </gazebo>
+    </gazebo>    -->
     <!-- Load Gazebo lib and set the robot namespace -->
     <gazebo>

File: iiwa_description/urdf/iiwa7.xacro (robot description, xacro)
@@ -274,5 +274,6 @@
         <origin xyz="0 0 -0.0005" rpy="0 0 0"/>
         <geometry>
-          <mesh filename="package://iiwa_description/meshes/iiwa7/visual/link_7.stl"/>
+          <!-- <mesh filename="package://iiwa_description/meshes/iiwa7/visual/link_7.stl"/> -->
+          <mesh filename="package://iiwa_description/meshes/iiwa7/visual/MF_Touch_pneumatisch.dae"/>
         </geometry>
         <material name="Grey"/>
@@ -281,5 +282,6 @@
         <origin xyz="0 0 -0.0005" rpy="0 0 0"/>
         <geometry>
-          <mesh filename="package://iiwa_description/meshes/iiwa7/collision/link_7.stl"/>
+          <!-- <mesh filename="package://iiwa_description/meshes/iiwa7/visual/link_7.stl"/> -->
+          <mesh filename="package://iiwa_description/meshes/iiwa7/visual/MF_Touch_pneumatisch.dae"/>
         </geometry>
         <material name="Grey"/>
@@ -289,7 +291,29 @@
       <parent link="${robot_name}_link_7"/>
       <child link="${robot_name}_link_ee"/>
-      <origin xyz="0 0 0.045" rpy="0 0 0"/>
+      <!-- <origin xyz="0 0 0.045" rpy="0 0 0"/> -->
+      <origin xyz="0 0 0.071" rpy="0 0 0"/> <!--0.045-->
     </joint>
     <link name="${robot_name}_link_ee">
+    <visual>
+        <origin xyz="0 0 0" rpy="${PI / 2} 0 0"/>
+        <geometry>
+          <mesh filename="package://iiwa_description/meshes/iiwa7/visual/tool_pneumatisch.dae"/>
+        </geometry>
+        <material name="Grey"/>
+      </visual>
+      <collision>
+        <origin xyz="0 0 0" rpy="${PI / 2} 0 0"/>
+        <geometry>
+          <mesh filename="package://iiwa_description/meshes/iiwa7/collision/tool_pneumatisch.dae"/>
+        </geometry>
+        <material name="Grey"/>
+      </collision>
+    </link>
+    <joint name="${robot_name}_joint_tool" type="fixed">
+      <parent link="${robot_name}_link_ee"/>
+      <child link="${robot_name}_link_tool"/>
+      <origin xyz="0 0 0" rpy="${PI} 0 ${PI}"/>
+    </joint>
+    <link name="${robot_name}_link_tool">
     </link>
     <!--Extensions -->
